File: embedded/hardware_2.0/rev_1.0/mcu_board/main.brd (EAGLE design)
At the start: 53.3 x 50.2 mm, 38 parts, among them IC1 MCP1703CB, Q1 8MHz

Commit message: aeris_2.0
Parts:
- added BOOT: (no value), jumper:JP1
- added C27, C28: 4.7uF, resistor:C0805
- added C29: 100n, resistor:C0805
- added C30, C31: 10uF, resistor:C0805
- added LED1: (no value), led:CHIPLED_1206
- added R4, R6, R7, R8, R9: 47k, resistor:M0805
- added R5: 330, resistor:M0805
- added S1, S2: DTSM-6, switch-tact:DTSM-6
- added SV1: programming, con-lstb:MA04-1
- added U$1: MICROSD, adafruit:MICROSD
- added WIFI: (no value), con-lstb:MA04-2
- moved C19 12.8 mm to (3.86, 46.7), turned to 0 degrees
- moved LED12 8.75 mm to (15.3, 3.00), turned to 180 degrees
- moved R27 5.89 mm to (15.2, 7.52), turned to 270 degrees
- moved C26 5.40 mm to (8.74, 47.1)
- moved C25 4.48 mm to (12.4, 47.1), turned to 180 degrees
- moved R13 3.07 mm to (48.0, 11.5)
- moved R14 3.05 mm to (45.5, 11.5)
- moved C8 2.19 mm to (5.89, 12.4)
- moved C13 1.63 mm to (46.7, 21.7)
- moved C9 1.55 mm to (37.6, 12.4)
- moved C18 1.42 mm to (16.9, 41.0), turned to 0 degrees
- moved CN1 1.42 mm to (7.92, 3.66)
- moved C24 1.22 mm to (37.8, 42.7)
- moved C10 0.45 mm to (40.4, 16.3)
Connections:
- removed net VCAP_1: IC_1.P$81
- removed net VCAP_2: IC_1.P$125
- new net KEY: IC_1.P$94, R8.1, S2.4
- new net LED: IC_1.P$95, R5.1
- new net N$13: IC_1.P$171, R9.2
- new net N$14: IC_1.P$1, IC_1.P$176
- new net N$5: C27.2, IC_1.P$81
- new net N$6: C28.2, IC_1.P$125
- new net N$7: LED1.A, R5.2
- new net N$8: R6.1, WIFI.6
- new net N$9: BOOT.1, IC_1.P$166, R7.2
- new net UART_RX: IC_1.P$121, WIFI.8
- new net UART_TX: IC_1.P$120, WIFI.1
- new net WIFI_RST: IC_1.P$119, WIFI.4
- net +3V3: now also BOOT.2, C30.1, C31.1, R4.2, R6.2, R8.2, U$1.4, WIFI.2
- net GND: now also C27.1, C28.1, C29.1, C30.2, C31.2, IC_1.P$58, LED1.C, R7.1, R9.1, S1.2, S2.2, SV1.3, U$1.6, U$1.MT1, U$1.MT2, WIFI.7
- net RESET: now also C29.2, IC_1.P$31, R4.1, S1.4, SV1.1; no longer EXPANSION.7
- net SWCLK: now also IC_1.P$137, SV1.4; no longer EXPANSION.1
- net SWDIO: now also IC_1.P$124, SV1.2; no longer EXPANSION.5
Routing:
- net +3V3: track 0.00 -> 313.3 mm, vias 0 -> 18
- net GND: track 0.00 -> 310.0 mm, vias 0 -> 18
- net RESET: track 0.00 -> 70.0 mm, vias 0 -> 5
- net UART_RX: track 0.00 -> 49.9 mm
- net SWCLK: track 0.00 -> 48.9 mm, vias 0 -> 1
- net WIFI_RST: track 0.00 -> 45.3 mm
- net UART_TX: track 0.00 -> 41.5 mm, vias 0 -> 2
- net N$9: track 0.00 -> 30.3 mm
- net N$4: track 0.00 -> 20.2 mm
- net LED: track 0.00 -> 19.5 mm
- net N$3: track 0.00 -> 18.0 mm
- net KEY: track 0.00 -> 16.7 mm
- net SWDIO: track 0.00 -> 16.5 mm
- net SDA: track 0.00 -> 10.7 mm
- net SCL: track 0.00 -> 9.87 mm
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