File: embedded/hardware_2.0/rev_1.0/mcu_board/main.sch (EAGLE design)
At the start: 38 parts, among them IC1 MCP1703CB, Q1 8MHz

Commit message: aeris_2.0
Parts:
- added BOOT: (no value), jumper:JP1E
- added C27, C28: 4.7uF, resistor:C-EUC0805
- added C29: 100n, resistor:C-EUC0805
- added C30, C31: 10uF, resistor:C-EUC0805
- added LED1: (no value), led:LEDCHIPLED_1206
- added R4, R6, R7, R8, R9: 47k, resistor:R-EU_M0805
- added R5: 330, resistor:R-EU_M0805
- added S1, S2: DTSM-6, switch-tact:DTSM-6
- added SV1: programming, con-lstb:MA04-1
- added U$1: MICROSD, adafruit:MICROSD
- added WIFI: (no value), con-lstb:MA04-2
Connections:
- new net KEY: IC_1.PB14, R8.1, S2.4
- new net LED: IC_1.PB15, R5.1
- new net N$13: IC_1.PDR_ON, R9.2
- new net N$14: IC_1.PE2, IC_1.PI7
- new net N$5: C27.2, IC_1.VCAP_1
- new net N$6: C28.2, IC_1.VCAP_2
- new net N$7: LED1.A, R5.2
- new net N$8: R6.1, WIFI.6
- new net N$9: BOOT.1, IC_1.BOOT_0, R7.2
- new net UART_RX: IC_1.PA10, WIFI.8
- new net UART_TX: IC_1.PA9, WIFI.1
- new net WIFI_RST: IC_1.PA8, WIFI.4
- net +3V3: now also BOOT.2, C30.1, C31.1, R4.2, R6.2, R8.2, U$1.VDD, WIFI.2
- net GND: now also C27.1, C28.1, C29.1, C30.2, C31.2, IC_1.PB2/BOOT_1, LED1.C, R7.1, R9.1, S1.2, S2.2, SV1.3, U$1.GND, U$1.GND1, U$1.VSS, WIFI.7
- net RESET: now also C29.2, IC_1.NRST, R4.1, S1.4, SV1.1; no longer EXPANSION.7
- net SWCLK: now also IC_1.PA14, SV1.4; no longer EXPANSION.1
- net SWDIO: now also IC_1.PA13, SV1.2; no longer EXPANSION.5
Other:
- moved on the sheet: C14, C19, C25, C26, Q1
